File: backplane/backplane.sch (EAGLE design)
At the start: 13 parts, among them U1 CDCLVC1104, U2 ASV-24.576MHZ-EJ-T, X1 PINCON-2X8, X5-JB PINCON-2X6, X5-JC PINCON-2X6, X5-JD PINCON-2X6, X5-JE PINCON-2X6, X5-JF PINCON-2X6

Commit message: added attributes to build a usable BOM
Parts:
- U2: MPN (none) -> ASV-24.576MHZ-EJ-T; OC_DIGIKEY (none) -> 535-9318-1-ND; OC_FARNELL (none) -> 1611834; OC_MOUSER (none) -> 815-ASV-24.576-EJ-T
