File: modules/headset_bottom_right/headset_br.brd (EAGLE design)
At the start: 100 x 62 mm, 287 parts, among them U1 CDCLVC1103, U2 2N7002, U3 2N7002, U300 ADAU1701/02ADAU1701JSTZ, U4 2N7002, U400 PGA2505, U5 2N7002, U500 PCM4202, U600 PCM1791A, U700 TPA6130A2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

Commit message: added attributes to build a usable BOM
Parts:
- LDO102: value LP2985 -> LP2985-50
- R37: value 480R -> 475R
