File: power/+49V/+49V.sch (EAGLE design)
At the start: 29 parts, among them U1 LM5001MAX, X1 PINCON-1X4, X2 PINCON-1X4

Commit message: added attributes to build a usable BOM
Parts:
- CBYP: MANUFACTURER (none) -> Murata; MPN (none) -> GRM155R61A105KE15D; OC_DIGIKEY (none) -> 490-3890-1-ND; OC_FARNELL (none) -> 1735523; OC_MOUSER (none) -> 81-GRM155R61A105KE15
- CIN1: MANUFACTURER (none) -> Murata; MPN (none) -> GRM216R71H103KA01D; OC_DIGIKEY (none) -> 490-1664-1-ND; OC_FARNELL (none) -> 1828948; OC_MOUSER (none) -> 81-GRM40X103K50D
- CIN2: MANUFACTURER (none) -> Kemet; MPN (none) -> C0805C104K5RACTU; OC_DIGIKEY (none) -> 399-1170-1-ND; OC_FARNELL (none) -> 2392344; OC_MOUSER (none) -> 80-C0805C104K5R
- CIN_1, CIN_2: MANUFACTURER (none) -> TDK; MPN (none) -> C3216X7R1H105K160AB; OC_DIGIKEY (none) -> 445-1423-1-ND; OC_FARNELL (none) -> 1907358; OC_MOUSER (none) -> 810-C3216X7R1H105K
- COUT: MANUFACTURER (none) -> TDK; MPN (none) -> C5750X7S2A106M; OC_DIGIKEY (none) -> 445-5212-1-ND; OC_FARNELL (none) -> 2112740; OC_MOUSER (none) -> 810-C5750X7S2A106M
- CSS: MANUFACTURER (none) -> Tayo Yuden; MPN (none) -> LMK212BJ106KG-T; OC_DIGIKEY (none) -> 587-1300-1-ND; OC_MOUSER (none) -> 963-LMK212BJ106KG-T
- RB: MANUFACTURER (none) -> Yageo; MPN (none) -> RC0805FR-076R8L; OC_DIGIKEY (none) -> 311-6.80CRCT-ND; OC_FARNELL (none) -> 9237224
