File: power/+6V/+6V.sch (EAGLE design)
At the start: 17 parts, among them U1 TPS54335, X1 PINCON-1X4, X2 PINCON-1X4

Commit message: added attributes to build a usable BOM
Parts:
- CIN: MANUFACTURER (none) -> TDK; MPN (none) -> C3225X5R1E106K; OC_DIGIKEY (none) -> 445-3946-1-ND; OC_FARNELL (none) -> 2346957; OC_MOUSER (none) -> 810-C3225X5R1E106K
- COUT: MANUFACTURER (none) -> TDK; MPN (none) -> C4532X5R1A476M; OC_DIGIKEY (none) -> 445-1440-1-ND; OC_FARNELL (none) -> 2112732; OC_MOUSER (none) -> 810-C4532X5R1A476M
