File: power/-6V/-6V.brd (EAGLE design)
At the start: 35.6 x 14 mm, 25 parts, among them U1 LM5575, X1 PINCON-1X4, X2 PINCON-1X4

Commit message: added attributes to build a usable BOM
Parts:
- RFBB: value (none) -> 1K65
- RFBT: value (none) -> 6K49
